Commit message: Added Gazebo launch files, working on camera integration. Need to migrate to new version of Gazebo

File: install/arduinobot_description/share/arduinobot_description/urdf/arduinobot.urdf.xacro (robot description, xacro)
@@ -4,6 +4,15 @@
     <xacro:property name="effort" value="30.0"/>
     <xacro:property name="velocity" value="10.0"/>
+    <xacro:macro name="default_inertial" params="mass">
+        <inertial>
+            <mass value="${mass}"/>
+            <inertia ixx="1.0" ixy="0.0" ixz="0.0"
+                     iyy="1.0" iyz="0.0"
+                     izz="1.0"/>
+        </inertial>
+    </xacro:macro>
     <link name="world"/>
     <link name="base_link">
+        <xacro:default_inertial mass="1.0"/>
         <visual>
             <origin rpy="0 0 0" xyz="-0.5 -0.5 0"/>
@@ -12,4 +21,10 @@
             </geometry>
         </visual>
+        <collision>
+            <origin rpy="0 0 0" xyz="-0.5 -0.5 0"/>
+            <geometry>
+                <mesh filename="package://arduinobot_description/meshes/basement.STL" scale="0.01 0.01 0.01"/>
+            </geometry>
+        </collision>
     </link>
     <joint name="virtual_joint" type="fixed">
@@ -19,4 +34,5 @@
     </joint>
     <link name="base_plate">
+        <xacro:default_inertial mass="0.1"/>
         <visual>
             <origin rpy="0 0 0" xyz="-0.39 -0.39 -0.56"/>
@@ -25,4 +41,10 @@
             </geometry>
         </visual>
+        <collision>
+            <origin rpy="0 0 0" xyz="-0.39 -0.39 -0.56"/>
+            <geometry>
+                <mesh filename="package://arduinobot_description/meshes/base_plate.STL" scale="0.01 0.01 0.01"/>
+            </geometry>
+        </collision>
     </link>
     <joint name="joint_1" type="revolute">
@@ -34,4 +56,5 @@
     </joint>
     <link name="forward_drive_arm">
+        <xacro:default_inertial mass="0.1"/>
         <visual>
             <origin rpy="0 -${PI/2} ${PI/2}" xyz="0.19 0.06 -0.08"/>
@@ -40,4 +63,10 @@
             </geometry>
         </visual>
+        <collision>
+            <origin rpy="0 -${PI/2} ${PI/2}" xyz="0.19 0.06 -0.08"/>
+            <geometry>
+                <mesh filename="package://arduinobot_description/meshes/forward_drive_arm.STL" scale="0.01 0.01 0.01"/>
+            </geometry>
+        </collision>
     </link>
     <joint name="joint_2" type="revolute">
@@ -49,4 +78,5 @@
     </joint>
     <link name="horizontal_arm">
+        <xacro:default_inertial mass="0.1"/>
         <visual>
             <origin rpy="${PI/2} 0 ${PI/2}" xyz="-0.03 -0.4 -0.06"/>
@@ -55,4 +85,10 @@
             </geometry>
         </visual>
+        <collision>
+            <origin rpy="${PI/2} 0 ${PI/2}" xyz="-0.03 -0.4 -0.06"/>
+            <geometry>
+                <mesh filename="package://arduinobot_description/meshes/horizontal_arm.STL" scale="0.01 0.01 0.01"/>
+            </geometry>
+        </collision>
     </link>
     <joint name="joint_3" type="revolute">
@@ -64,4 +100,5 @@
     </joint>
     <link name="claw_support">
+        <xacro:default_inertial mass="0.05"/>
         <visual>
             <origin rpy="0 0 ${PI/2}" xyz="0 -0.05 -0.15"/>
@@ -70,4 +107,10 @@
             </geometry>
         </visual>
+        <collision>
+            <origin rpy="0 0 ${PI/2}" xyz="0 -0.05 -0.15"/>
+            <geometry>
+                <mesh filename="package://arduinobot_description/meshes/claw_support.STL" scale="0.01 0.01 0.01"/>
+            </geometry>
+        </collision>
     </link>
     <joint name="horizontal_arm_to_claw_support" type="fixed">
@@ -77,4 +120,5 @@
     </joint>
     <link name="gripper_right">
+        <xacro:default_inertial mass="0.01"/>
         <visual>
             <origin xyz="-0.1 0.5 -0.1" rpy="0 0 -${PI/2}"/>
@@ -83,6 +127,13 @@
             </geometry>
         </visual>
+        <collision>
+            <origin xyz="-0.1 0.5 -0.1" rpy="0 0 -${PI/2}"/>
+            <geometry>
+                <mesh filename="package://arduinobot_description/meshes/right_finger.STL" scale="0.01 0.01 0.01"/>
+            </geometry>
+        </collision>
     </link>
     <link name="gripper_left">
+        <xacro:default_inertial mass="0.01"/>
         <visual>
             <origin xyz="-0.04 0.5 -0.1" rpy="0 0 -${PI/2}"/>
@@ -91,4 +142,10 @@
             </geometry>
         </visual>
+        <collision>
+            <origin xyz="-0.04 0.5 -0.1" rpy="0 0 -${PI/2}"/>
+            <geometry>
+                <mesh filename="package://arduinobot_description/meshes/left_finger.STL" scale="0.01 0.01 0.01"/>
+            </geometry>
+        </collision>
     </link>
     <joint name="joint_4" type="revolute">
@@ -107,3 +164,59 @@
         <limit lower="0.0" upper="${PI/2}" effort="${effort}" velocity="${velocity}"/>
     </joint>
+    <link name="rgb_camera">
+        <xacro:default_inertial mass="0.001"/>
+        <visual>
+            <origin rpy="-1.57 0 -1.57" xyz="-0.1 0.125 0.15"/>
+            <geometry>
+                <mesh filename="package://arduinobot_description/meshes/pi_camera.STL" scale="0.01 0.01 0.01"/>
+            </geometry>
+        </visual>
+        <collision>
+            <origin xyz="-0.04 0.5 -0.1" rpy="0 0 -${PI/2}"/>
+            <geometry>
+                <mesh filename="package://arduinobot_description/meshes/left_finger.STL" scale="0.01 0.01 0.01"/>
+            </geometry>
+        </collision>
+    </link>
+    <joint name="rgb_camera_joint" type="fixed">
+        <parent link="base_link"/>
+        <child link="rgb_camera"/>
+        <origin rpy="0 -0.5 1.57" xyz="0 0.45 0.2"/>
+    </joint>
+    <gazebo reference="rgb_camera">
+        <sensor name="camera" type="camera">
+            <always_on>true</always_on>
+            <update_rate>30.0</update_rate>
+            <visualize>true</visualize>
+            <topic>/image_raw</topic>
+            <gz_frame_id>/rgb_camera</gz_frame_id>
+            <camera name="camera">
+                <horizontal_fov>1.21126</horizontal_fov>
+                <image>
+                    <width>2304</width>
+                    <height>1296</height>
+                    <format>R8G8B8</format>
+                </image>
+                <distortion>
+                    <k1>0.0</k1>
+                    <k2>0.0</k2>
+                    <k3>0.0</k3>
+                    <p1>0.0</p1>
+                    <p2>0.0</p2>
+                    <center>0.5 0.5</center>
+                </distortion>
+            </camera>
+        </sensor>
+    </gazebo>
+    <gazebo>
+        <!-- ROS 2 Iron or above -->
+        <xacro:unless value="$(arg is_ignition)">
+            <plugin filename="gz_ros2_control-system" name="gz_ros2_control::GazeboSimROS2ControlPlugin">
+            <parameters>$(find arduinobot_controller)/config/arduinobot_controllers.yaml</parameters>
+            </plugin>
+            <plugin filename="gz-sim-sensors-system" name="gz::sim::systems::Sensors">
+            <render_engine>ogre2</render_engine>
+            </plugin>
+        </xacro:unless>
+    </gazebo>
 </robot>

Commit message: Working rgb-camera sensor

File: install/arduinobot_description/share/arduinobot_description/urdf/arduinobot.urdf.xacro (robot description, xacro)
@@ -1,4 +1,5 @@
 <?xml version="1.0"?>
 <robot xmlns:xacro="http://www.ros.org/wiki/xacro" name="arduinobot">
+    <xacro:arg name="is_ignition" default="false"/>
     <xacro:property name="PI" value="3.14159"/>
     <xacro:property name="effort" value="30.0"/>
@@ -175,5 +176,5 @@
             <origin xyz="-0.04 0.5 -0.1" rpy="0 0 -${PI/2}"/>
             <geometry>
-                <mesh filename="package://arduinobot_description/meshes/left_finger.STL" scale="0.01 0.01 0.01"/>
+                <mesh filename="package://arduinobot_description/meshes/pi_camera.STL" scale="0.01 0.01 0.01"/>
             </geometry>
         </collision>
@@ -210,13 +211,7 @@
     </gazebo>
     <gazebo>
-        <!-- ROS 2 Iron or above -->
-        <xacro:unless value="$(arg is_ignition)">
-            <plugin filename="gz_ros2_control-system" name="gz_ros2_control::GazeboSimROS2ControlPlugin">
-            <parameters>$(find arduinobot_controller)/config/arduinobot_controllers.yaml</parameters>
-            </plugin>
-            <plugin filename="gz-sim-sensors-system" name="gz::sim::systems::Sensors">
+        <plugin filename="ignition-gazebo-sensors-system" name="ignition::gazebo::systems::Sensors">
             <render_engine>ogre2</render_engine>
-            </plugin>
-        </xacro:unless>
+        </plugin>
     </gazebo>
 </robot>
