Commit message: Ported over and fixed issues with original code.

File: install/arduinobot_description/share/arduinobot_description/urdf/arduinobot.urdf.xacro (robot description, xacro)
@@ -1,22 +1,25 @@
 <?xml version="1.0"?>
 <robot xmlns:xacro="http://www.ros.org/wiki/xacro" name="arduinobot">
+    <!-- Start GZ or Ignition depending on ROS 2 Version -->
     <xacro:arg name="is_ignition" default="true"/>
-    <!-- <xacro:arg name="gazebo_xacro_file" default="urdf/arduinobot_gazebo.xacro"/>
-    <xacro:include filename="${gazebo_xacro_file}"/> -->
-    <!-- <xacro:include filename="${find arduinobot_description)/urdf/arduinobot_gazebo.xacro"/>
-    <xacro:include filename="${find arduinobot_description)/urdf/arduinobot_ros2_control.xacro"/> -->
-    <xacro:include filename="$(find arduinobot_description)/urdf/arduinobot_gazebo.xacro"/>
-    <xacro:include filename="$(find arduinobot_description)/urdf/arduinobot_ros2_control.xacro"/>
-    <xacro:property name="PI" value="3.14159"/>
-    <xacro:property name="effort" value="30.0"/>
-    <xacro:property name="velocity" value="10.0"/>
+    <!-- Include Gazebo Parameters -->
+    <xacro:include filename="$(find arduinobot_description)/urdf/arduinobot_gazebo.xacro" />
+    <!-- Include ros2_control Plugins -->
+    <xacro:include filename="$(find arduinobot_description)/urdf/arduinobot_ros2_control.xacro" />
+    <!-- Useful XACRO Variables (Properties) -->
+    <xacro:property name="PI" value="3.14159265359" />
+    <xacro:property name="effort" value="30.0" />
+    <xacro:property name="velocity" value="10.0" />
+    <!-- Useful Macros -->
     <xacro:macro name="default_inertial" params="mass">
         <inertial>
-            <mass value="${mass}"/>
+            <origin xyz="0 0 0" rpy="0 0 0"/>
+            <mass value="${mass}" />
             <inertia ixx="1.0" ixy="0.0" ixz="0.0"
                      iyy="1.0" iyz="0.0"
-                     izz="1.0"/>
+                     izz="1.0" />
         </inertial>
     </xacro:macro>
+    <!-- Links -->
     <link name="world"/>
     <link name="base_link">
@@ -35,9 +38,4 @@
         </collision>
     </link>
-    <joint name="virtual_joint" type="fixed">
-        <parent link="world"/>
-        <child link="base_link"/>
-        <origin rpy="0 0 0" xyz="0 0 0"/>
-    </joint>
     <link name="base_plate">
         <xacro:default_inertial mass="0.1"/>
@@ -55,15 +53,8 @@
         </collision>
     </link>
-    <joint name="joint_1" type="revolute">
-        <parent link="base_link"/>
-        <child link="base_plate"/>
-        <axis xyz="0 0 1"/>
-        <origin rpy="0 0 0" xyz="0 0 0.307"/>
-        <limit lower="-${PI/2}" upper="${PI/2}" effort="${effort}" velocity="${velocity}"/>
-    </joint>
     <link name="forward_drive_arm">
         <xacro:default_inertial mass="0.1"/>
         <visual>
-            <origin rpy="0 -${PI/2} ${PI/2}" xyz="0.19 0.06 -0.08"/>
+            <origin rpy=" 0 -${PI / 2} ${PI / 2}" xyz="0.19 0.06 -0.08"/>
             <geometry>
                 <mesh filename="package://arduinobot_description/meshes/forward_drive_arm.STL" scale="0.01 0.01 0.01"/>
@@ -71,5 +62,5 @@
         </visual>
         <collision>
-            <origin rpy="0 -${PI/2} ${PI/2}" xyz="0.19 0.06 -0.08"/>
+            <origin rpy=" 0 -${PI / 2} ${PI / 2}" xyz="0.19 0.06 -0.08"/>
             <geometry>
                 <mesh filename="package://arduinobot_description/meshes/forward_drive_arm.STL" scale="0.01 0.01 0.01"/>
@@ -77,15 +68,8 @@
         </collision>
     </link>
-    <joint name="joint_2" type="revolute">
-        <parent link="base_plate"/>
-        <child link="forward_drive_arm"/>
-        <axis xyz="1 0 0"/>
-        <origin rpy="0 0 0" xyz="-0.02 0 0.35"/>
-        <limit lower="-${PI/2}" upper="${PI/2}" effort="${effort}" velocity="${velocity}"/>
-    </joint>
     <link name="horizontal_arm">
         <xacro:default_inertial mass="0.1"/>
         <visual>
-            <origin rpy="${PI/2} 0 ${PI/2}" xyz="-0.03 -0.4 -0.06"/>
+            <origin rpy="${PI / 2} 0 ${PI / 2}" xyz="-0.03 -0.4 -0.06"/>
             <geometry>
                 <mesh filename="package://arduinobot_description/meshes/horizontal_arm.STL" scale="0.01 0.01 0.01"/>
@@ -93,5 +77,5 @@
         </visual>
         <collision>
-            <origin rpy="${PI/2} 0 ${PI/2}" xyz="-0.03 -0.4 -0.06"/>
+            <origin rpy="${PI / 2} 0 ${PI / 2}" xyz="-0.03 -0.4 -0.06"/>
             <geometry>
                 <mesh filename="package://arduinobot_description/meshes/horizontal_arm.STL" scale="0.01 0.01 0.01"/>
@@ -99,15 +83,8 @@
         </collision>
     </link>
-    <joint name="joint_3" type="revolute">
-        <parent link="forward_drive_arm"/>
-        <child link="horizontal_arm"/>
-        <axis xyz="1 0 0"/>
-        <origin rpy="0 0 0" xyz="0 0 0.8"/>
-        <limit lower="-${PI/2}" upper="${PI/2}" effort="${effort}" velocity="${velocity}"/>
-    </joint>
     <link name="claw_support">
         <xacro:default_inertial mass="0.05"/>
         <visual>
-            <origin rpy="0 0 ${PI/2}" xyz="0 -0.05 -0.15"/>
+            <origin rpy="0 0 ${PI / 2}" xyz="0 -0.05 -0.15"/>
             <geometry>
                 <mesh filename="package://arduinobot_description/meshes/claw_support.STL" scale="0.01 0.01 0.01"/>
@@ -115,5 +92,5 @@
         </visual>
         <collision>
-            <origin rpy="0 0 ${PI/2}" xyz="0 -0.05 -0.15"/>
+            <origin rpy="0 0 ${PI / 2}" xyz="0 -0.05 -0.15"/>
             <geometry>
                 <mesh filename="package://arduinobot_description/meshes/claw_support.STL" scale="0.01 0.01 0.01"/>
@@ -121,13 +98,8 @@
         </collision>
     </link>
-    <joint name="horizontal_arm_to_claw_support" type="fixed">
-        <parent link="horizontal_arm"/>
-        <child link="claw_support"/>
-        <origin xyz="0 0.82 0" rpy="0 0 0"/>
-    </joint>
     <link name="gripper_right">
         <xacro:default_inertial mass="0.01"/>
         <visual>
-            <origin xyz="-0.1 0.5 -0.1" rpy="0 0 -${PI/2}"/>
+            <origin rpy="0 0 -${PI / 2}" xyz="-0.1 0.50 -0.1"/>
             <geometry>
                 <mesh filename="package://arduinobot_description/meshes/right_finger.STL" scale="0.01 0.01 0.01"/>
@@ -135,5 +107,5 @@
         </visual>
         <collision>
-            <origin xyz="-0.1 0.5 -0.1" rpy="0 0 -${PI/2}"/>
+            <origin rpy="0 0 -${PI / 2}" xyz="-0.1 0.50 -0.1"/>
             <geometry>
                 <mesh filename="package://arduinobot_description/meshes/right_finger.STL" scale="0.01 0.01 0.01"/>
@@ -144,5 +116,5 @@
         <xacro:default_inertial mass="0.01"/>
         <visual>
-            <origin xyz="-0.04 0.5 -0.1" rpy="0 0 -${PI/2}"/>
+            <origin rpy="0 0 -${PI / 2}" xyz="-0.04 0.50 -0.1"/>
             <geometry>
                 <mesh filename="package://arduinobot_description/meshes/left_finger.STL" scale="0.01 0.01 0.01"/>
@@ -150,5 +122,5 @@
         </visual>
         <collision>
-            <origin xyz="-0.04 0.5 -0.1" rpy="0 0 -${PI/2}"/>
+            <origin rpy="0 0 -${PI / 2}" xyz="-0.04 0.50 -0.1"/>
             <geometry>
                 <mesh filename="package://arduinobot_description/meshes/left_finger.STL" scale="0.01 0.01 0.01"/>
@@ -156,90 +128,55 @@
         </collision>
     </link>
-    <joint name="joint_4" type="revolute">
+    <!-- Joints -->
+    <joint name="virtual_joint" type="fixed">
+        <parent link="world"/>
+        <child link="base_link"/>
+        <origin xyz="0 0 0" rpy="0 0 0"/>
+    </joint>
+    <joint name ="joint_1" type="revolute">
+        <parent link="base_link"/>
+        <child link = "base_plate"/>
+        <origin xyz="0 0 0.307"/>
+        <axis xyz="0 0 1"/>
+        <limit lower="-${PI / 2}" upper="${PI / 2}"
+               effort="${effort}" velocity="${velocity}"/>
+    </joint>
+    <joint name ="joint_2" type="revolute">
+        <parent link="base_plate"/>
+        <child link = "forward_drive_arm"/>
+        <origin xyz="-0.02 0 0.35"/>
+        <axis xyz="1 0 0"/>
+        <limit lower="-${PI / 2}" upper="${PI / 2}"
+                effort="${effort}" velocity="${velocity}"/>
+    </joint>
+    <joint name ="joint_3" type="revolute">
+        <parent link="forward_drive_arm"/>
+        <child link = "horizontal_arm"/>
+        <origin xyz="0 0 0.8"/>
+        <axis xyz="1 0 0"/>
+        <limit lower="-${PI / 2}" upper="${PI / 2}"
+               effort="${effort}" velocity="${velocity}"/>
+    </joint>
+    <joint name ="horizontal_arm_to_claw_support" type="fixed">
+        <parent link="horizontal_arm"/>
+        <child link = "claw_support"/>
+        <origin xyz="0 0.82 0"/>
+    </joint>
+    <joint name ="joint_4" type="revolute">
         <parent link="claw_support"/>
-        <child link="gripper_right"/>
+        <child link = "gripper_right"/>
+        <origin xyz="-0.04 0.13 -0.1"/>
         <axis xyz="0 0 1"/>
-        <origin rpy="0 0 0" xyz="-0.04 0.13 -0.1"/>
-        <limit lower="-${PI/2}" upper="0.0" effort="${effort}" velocity="${velocity}"/>
+        <limit lower="-${PI / 2}" upper="0.0"
+               effort="${effort}" velocity="${velocity}"/>
     </joint>
-    <joint name="joint_5" type="revolute">
+    <joint name ="joint_5" type="revolute">
         <parent link="claw_support"/>
-        <child link="gripper_left"/>
+        <child link = "gripper_left"/>
+        <origin xyz="-0.22 0.13 -0.1"/>
         <axis xyz="0 0 1"/>
-        <origin rpy="0 0 0" xyz="-0.22 0.13 -0.1"/>
+        <limit lower="0.0" upper="${PI / 2}"
+               effort="${effort}" velocity="${velocity}"/>
         <mimic joint="joint_4" multiplier="-1"/>
-        <limit lower="0.0" upper="${PI/2}" effort="${effort}" velocity="${velocity}"/>
     </joint>
-    <link name="rgb_camera">
-        <xacro:default_inertial mass="0.001"/>
-        <visual>
-            <origin rpy="-1.57 0 -1.57" xyz="-0.1 0.125 0.15"/>
-            <geometry>
-                <mesh filename="package://arduinobot_description/meshes/pi_camera.STL" scale="0.01 0.01 0.01"/>
-            </geometry>
-        </visual>
-        <collision>
-            <origin xyz="-0.04 0.5 -0.1" rpy="0 0 -${PI/2}"/>
-            <geometry>
-                <mesh filename="package://arduinobot_description/meshes/pi_camera.STL" scale="0.01 0.01 0.01"/>
-            </geometry>
-        </collision>
-    </link>
-    <joint name="rgb_camera_joint" type="fixed">
-        <parent link="base_link"/>
-        <child link="rgb_camera"/>
-        <origin rpy="0 -0.5 1.57" xyz="0 0.45 0.2"/>
-    </joint>
-    <gazebo reference="rgb_camera">
-        <sensor name="camera" type="camera">
-            <always_on>true</always_on>
-            <update_rate>30.0</update_rate>
-            <visualize>true</visualize>
-            <topic>/image_raw</topic>
-            <gz_frame_id>/rgb_camera</gz_frame_id>
-            <camera name="camera">
-                <horizontal_fov>1.21126</horizontal_fov>
-                <image>
-                    <width>2304</width>
-                    <height>1296</height>
-                    <format>R8G8B8</format>
-                </image>
-                <distortion>
-                    <k1>0.0</k1>
-                    <k2>0.0</k2>
-                    <k3>0.0</k3>
-                    <p1>0.0</p1>
-                    <p2>0.0</p2>
-                    <center>0.5 0.5</center>
-                </distortion>
-            </camera>
-        </sensor>
-    </gazebo>
-<gazebo>
-  <!-- ROS 2 Humble -->
-  <xacro:if value="$(arg is_ignition)">
-    <plugin filename="ign_ros2_control-system" name="ign_ros2_control::IgnitionROS2ControlPlugin">
-      <parameters>$(find arduinobot_controller)/config/arduinobot_controllers.yaml</parameters>
-    </plugin>
-    <plugin filename="ignition-gazebo-sensors-system" name="ignition::gazebo::systems::Sensors">
-      <render_engine>ogre2</render_engine>
-    </plugin>
-  </xacro:if>
-  <!-- ROS 2 Iron or above -->
-  <xacro:unless value="$(arg is_ignition)">
-    <plugin filename="gz_ros2_control-system" name="gz_ros2_control::GazeboSimROS2ControlPlugin">
-      <parameters>$(find arduinobot_controller)/config/arduinobot_controllers.yaml</parameters>
-    </plugin>
-    <plugin filename="gz-sim-sensors-system" name="gz::sim::systems::Sensors">
-      <render_engine>ogre2</render_engine>
-    </plugin>
-  </xacro:unless>
-</gazebo>
-<!--
-    <gazebo>
-        <plugin filename="ignition-gazebo-sensors-system" name="ignition::gazebo::systems::Sensors">
-            <render_engine>ogre2</render_engine>
-        </plugin>
-    </gazebo>
- -->
 </robot>

File: install/arduinobot_description/share/arduinobot_description/urdf/arduinobot_gazebo.xacro (robot description, xacro)
@@ -1,16 +1,18 @@
 <?xml version="1.0"?>
 <robot xmlns:xacro="http://www.ros.org/wiki/xacro" name="arduinobot">
-<!-- <xacro:arg name="controller_config" default="config/arduinobot_controllers.yaml"/> -->
-    <gazebo>
-        <xacro:if value="$(arg is_ignition)">
-            <plugin filename="ign_ros2_control-system" name="ign_ros2_control::IgnitionROS2ControlPlugin">
-                <parameters>$(find arduinobot_controller)/config/arduinobot_controllers.yaml</parameters>
-            </plugin>
-        </xacro:if>
-        <xacro:unless value="$(arg is_ignition)">
-            <plugin filename="gz_ros2_control-system" name="gz_ros2_control::GazeboSimROS2ControlPlugin">
-                <parameters>$(find arduinobot_controller)/config/arduinobot_controllers.yaml</parameters>
-            </plugin>
-        </xacro:unless>
-    </gazebo>
+  <!-- ROS 2 Control -->
+  <gazebo>
+    <!-- ROS 2 Humble -->
+    <xacro:if value="$(arg is_ignition)">
+      <plugin filename="ign_ros2_control-system" name="ign_ros2_control::IgnitionROS2ControlPlugin">
+        <parameters>$(find arduinobot_controller)/config/arduinobot_controllers.yaml</parameters>
+      </plugin>
+    </xacro:if>
+    <!-- ROS 2 Iron or above -->
+    <xacro:unless value="$(arg is_ignition)">
+      <plugin filename="gz_ros2_control-system" name="gz_ros2_control::GazeboSimROS2ControlPlugin">
+        <parameters>$(find arduinobot_controller)/config/arduinobot_controllers.yaml</parameters>
+      </plugin>
+    </xacro:unless>
+  </gazebo>
 </robot>

File: install/arduinobot_description/share/arduinobot_description/urdf/arduinobot_ros2_control.xacro (robot description, xacro)
@@ -1,6 +1,8 @@
 <?xml version="1.0"?>
 <robot xmlns:xacro="http://www.ros.org/wiki/xacro" name="arduinobot">
-    <xacro:property name="PI" value="3.14159"/>
-    <ros2_control type="system" name="RobotSystem">
+    <ros2_control name="RobotSystem" type="system">
+        <xacro:property name="PI" value="3.14159265359" />
+        <!-- ros2_control Gazebo -->
+        <!-- ROS 2 Humble -->
         <xacro:if value="$(arg is_ignition)">
             <hardware>
@@ -8,4 +10,5 @@
             </hardware>
         </xacro:if>
+        <!-- ROS 2 Iron or above -->
         <xacro:unless value="$(arg is_ignition)">
             <hardware>
@@ -15,6 +18,6 @@
         <joint name="joint_1">
             <command_interface name="position">
-                <param name="min">-${PI / 2}</param>
-                <param name="max">${PI / 2}</param>
+            <param name="min">-${PI / 2}</param>
+            <param name="max">${PI / 2}</param>
             </command_interface>
             <state_interface name="position"/>
@@ -22,6 +25,6 @@
         <joint name="joint_2">
             <command_interface name="position">
-                <param name="min">-${PI / 2}</param>
-                <param name="max">${PI / 2}</param>
+            <param name="min">-${PI / 2}</param>
+            <param name="max">${PI / 2}</param>
             </command_interface>
             <state_interface name="position"/>
@@ -29,6 +32,6 @@
         <joint name="joint_3">
             <command_interface name="position">
-                <param name="min">-${PI / 2}</param>
-                <param name="max">${PI / 2}</param>
+            <param name="min">-${PI / 2}</param>
+            <param name="max">${PI / 2}</param>
             </command_interface>
             <state_interface name="position"/>
@@ -36,6 +39,6 @@
         <joint name="joint_4">
             <command_interface name="position">
-                <param name="min">-${PI / 2}</param>
-                <param name="max">0.0</param>
+            <param name="min">-${PI / 2}</param>
+            <param name="max">0.0</param>
             </command_interface>
             <state_interface name="position"/>

Commit message: Just need robot control interface now

File: install/arduinobot_description/share/arduinobot_description/urdf/arduinobot.urdf.xacro (robot description, xacro)
@@ -1,4 +1,5 @@
 <?xml version="1.0"?>
 <robot xmlns:xacro="http://www.ros.org/wiki/xacro" name="arduinobot">
+    <xacro:arg name="is_sim" default="true"/>
     <!-- Start GZ or Ignition depending on ROS 2 Version -->
     <xacro:arg name="is_ignition" default="true"/>

File: install/arduinobot_description/share/arduinobot_description/urdf/arduinobot_ros2_control.xacro (robot description, xacro)
@@ -4,14 +4,26 @@
         <xacro:property name="PI" value="3.14159265359" />
         <!-- ros2_control Gazebo -->
-        <!-- ROS 2 Humble -->
-        <xacro:if value="$(arg is_ignition)">
+        <xacro:if value="${xacro.arg ('is_sim')}">
+            <!-- ROS 2 Humble -->
+            <xacro:if value="$(arg is_ignition)">
+                <hardware>
+                    <plugin>ign_ros2_control/IgnitionSystem</plugin>
+                </hardware>
+            </xacro:if>
+            <!-- ROS 2 Iron or above -->
+            <xacro:unless value="$(arg is_ignition)">
+                <hardware>
+                    <plugin>gz_ros2_control/GazeboSimSystem</plugin>
+                </hardware>
+            </xacro:unless>
+            <joint name="joint_5">
+                <param name="mimic">joint_4</param>
+                <param name="multiplier">-1</param>
+            </joint>
+        </xacro:if>
+        <xacro:unless value="${xacro.arg ('is_sim')}">
             <hardware>
-                <plugin>ign_ros2_control/IgnitionSystem</plugin>
-            </hardware>
-        </xacro:if>
-        <!-- ROS 2 Iron or above -->
-        <xacro:unless value="$(arg is_ignition)">
-            <hardware>
-                <plugin>gz_ros2_control/GazeboSimSystem</plugin>
+                <plugin>arduinobot_controller/ArduinobotInterface</plugin>
+                <param name="port">/dev/ttyACM0</param>
             </hardware>
         </xacro:unless>
@@ -44,8 +56,4 @@
             <state_interface name="position"/>
         </joint>
-        <joint name="joint_5">
-            <param name="mimic">joint_4</param>
-            <param name="multiplier">-1</param>
-        </joint>
     </ros2_control>
 </robot>
